File: zx_keyboard.sch (KiCad schematic (older format))
At the start: 3 parts, among them SW1 SW_PUSH, SW2 SW_PUSH, U1 4066

Commit message: kb
Parts:
- added D? (x4): D, symbol D
- added R1, R2, R3, R4, R5: 10K, symbol R
- added SW? (x38): SW_PUSH, Buttons_Switches_Keyboard:SW_Cherry_MX1A_1.00u_PCB, symbol SW_PUSH
Connections:
- net +3V3: now also R1.2, R2.2, R3.2, R4.2, R5.2; no longer U1.14 (V+)
- net at U1.1 (I/O): no longer U1.5 (ON)
- net at U1.13 (ON): no longer U1.2 (O/I)
- net at U1.14 (V+): no longer U1.3 (O/I)
- net at U1.14 (V+): no longer U1.10 (O/I)
- net at U1.4 (I/O): no longer SW2.2
- net at U1.14 (V+): no longer SW1.1
- net at U1.6 (ON): no longer U1.8 (I/O)
- net at U1.7 (V-): no longer U1.9 (O/I)
- net at SW1.2: now also SW2.2, SW?.2, SW?.2; no longer SW2.1
- new net: D?.2 (A), SW1.1, SW?.1, SW?.1, SW?.1, SW?.1
- new net: D?.2 (A), SW2.1, SW?.1, SW?.1, SW?.1, SW?.1
- new net: D?.2 (A), SW?.1, SW?.1, SW?.1, SW?.1, SW?.1
- new net: D?.2 (A), SW?.1, SW?.1, SW?.1, SW?.1
- new net: SW?.2, SW?.2, SW?.2, SW?.2 (x9)
Other:
- moved on the sheet: SW1, SW2, U1A, U1B, U1C, U1D

Commit message: kb
Parts:
- added D5, D6, D7, D8: D, symbol D
- SW1: value SW_PUSH -> KEY_1
- gave numbers to parts that had none: 42
- renumbered SW2 to SW11
Connections:
- net KD0: now also R1.1
- net at D1.2 (A), SW31.1, SW32.1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: now also SW35.1
- net at SW6.1: now also SW10.1, SW7.1, SW8.1, SW9.1, D5.2 (A)
- net at SW16.1: now also SW17.1, SW18.1, SW19.1, SW20.1, D6.2 (A)
- net at SW26.1: now also SW27.1, SW28.1, SW29.1, SW30.1, D7.2 (A)
- net at SW36.1: now also SW37.1, SW38.1, SW39.1, SW40.1, D8.2 (A)
Other:
- moved on the sheet: R1, R2, R3, R4, R5, SW10, SW12, SW13, SW14, SW15, SW16, SW17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

Commit message: kb
Parts:
- removed unit 2 of U1
- removed unit 3 of U1
- removed unit 4 of U1
- added C1: 10uF, symbol CP
- added D?: D, symbol D
- added P1: CONN_02X08, symbol CONN_02X08
- added R?: 1K, symbol R
- added R?: 10K, symbol R
- added SW41: KEY_CS2, Buttons_Switches_Keyboard:SW_Cherry_MX1A_1.00u_PCB, symbol SW_PUSH
- added SW42: KEY_SS2, Buttons_Switches_Keyboard:SW_Cherry_MX1A_1.00u_PCB, symbol SW_PUSH
- added SW43: KEY_TV, Buttons_Switches_Keyboard:SW_Cherry_MX1A_1.00u_PCB, symbol SW_PUSH
- SW10: value SW_PUSH -> KEY_0
- SW11: value SW_PUSH -> KEY_Q
- SW12: value SW_PUSH -> KEY_W
- SW13: value SW_PUSH -> KEY_E
- SW14: value SW_PUSH -> KEY_R
- SW15: value SW_PUSH -> KEY_T
- SW16: value SW_PUSH -> KEY_Y
- SW17: value SW_PUSH -> KEY_U
- SW18: value SW_PUSH -> KEY_I
- SW19: value SW_PUSH -> KEY_O
- SW2: value SW_PUSH -> KEY_2
- SW20: value SW_PUSH -> KEY_P
- SW21: value SW_PUSH -> KEY_A
- SW22: value SW_PUSH -> KEY_S
- SW23: value SW_PUSH -> KEY_D
- SW24: value SW_PUSH -> KEY_F
- SW25: value SW_PUSH -> KEY_G
- SW26: value SW_PUSH -> KEY_H
- SW27: value SW_PUSH -> KEY_J
- SW28: value SW_PUSH -> KEY_K
- SW29: value SW_PUSH -> KEY_L
- SW3: value SW_PUSH -> KEY_3
- SW30: value SW_PUSH -> KEY_EN
- SW31: value SW_PUSH -> KEY_CS1
- SW32: value SW_PUSH -> KEY_Z
- SW33: value SW_PUSH -> KEY_X
- SW34: value SW_PUSH -> KEY_C
- SW35: value SW_PUSH -> KEY_V
- SW36: value SW_PUSH -> KEY_B
- SW37: value SW_PUSH -> KEY_N
- SW38: value SW_PUSH -> KEY_M
- SW39: value SW_PUSH -> KEY_SS1
- SW4: value SW_PUSH -> KEY_4
- SW40: value SW_PUSH -> KEY_SP
- SW5: value SW_PUSH -> KEY_5
- SW6: value SW_PUSH -> KEY_6
- SW7: value SW_PUSH -> KEY_7
- SW8: value SW_PUSH -> KEY_8
- SW9: value SW_PUSH -> KEY_9
Connections:
- net +3V3: now also R1.1, R3.1, R4.1, R5.1, U1.14 (V+), C1.1, P1.14 (P14), SW43.1; no longer R1.2, R3.2, R4.2, R5.2
- net GND: now also U1.7 (V-), C1.2, P1.16 (P16), R?.2
- net KA10: now also D3.1 (K), P1.5 (P5)
- net KA11: now also D4.1 (K), P1.7 (P7)
- net KA12: now also D5.1 (K), P1.9 (P9)
- net KA13: now also D6.1 (K), P1.11 (P11)
- net KA14: now also D7.1 (K), P1.13 (P13)
- net KA15: now also D8.1 (K), P1.15 (P15)
- net KA8: now also D1.1 (K), P1.1 (P1)
- net KA9: now also D2.1 (K), P1.3 (P3)
- net KD0: now also R1.2, SW1.2, SW10.2, SW11.2, SW20.2, SW21.2, SW30.2, SW31.2, SW40.2, P1.2 (P2), SW41.2; no longer R1.1
- net KD1: now also R2.1, SW12.2, SW19.2, SW2.2, SW22.2, SW29.2, SW32.2, SW39.2, SW9.2, P1.4 (P4), SW42.2
- net KD2: now also R3.2, SW13.2, SW18.2, SW23.2, SW28.2, SW3.2, SW33.2, SW38.2, SW8.2, U1.1 (I/O), P1.6 (P6)
- net KD3: now also R4.2, SW14.2, SW17.2, SW24.2, SW27.2, SW34.2, SW37.2, SW4.2, SW7.2, P1.8 (P8)
- net KD4: now also R5.2, SW15.2, SW16.2, SW25.2, SW26.2, SW35.2, SW36.2, SW5.2, SW6.2, P1.10 (P10)
- net at U1.13 (ON): now also R?.1
- net DKA11: now reaches U1.2 (O/I)
- net DKA11: now also D4.2 (A), SW1.1, SW2.1, SW3.1, SW4.1, SW5.1
- net at D1.2 (A), SW31.1, SW32.1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: now also SW41.1
- net at D8.2 (A), SW36.1, SW37.1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: now also SW42.1
- new net: D?.2 (A), R?.1, R?.2, SW43.2
- new net CS_CTRL: D?.1 (K)
- no-connect marks 0 -> 1
Other:
- moved on the sheet: D1, D2, D3, D4, D5, D6, D7, D8, R1, R2, R3, R4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

Commit message: zx
Parts:
- added D? (x21): D, symbol D
- added R? (x16): 1K, symbol R
- added R? (x16): 10K, symbol R
- added SW? (x15): KEY_TV, Buttons_Switches_Keyboard:SW_Cherry_MX1A_1.00u_PCB, symbol SW_PUSH
- added U? (x16): 4066, TO_SOT_Packages_SMD:SOT-428, symbol 4066
Connections:
- net +3V3: now also SW?.1, SW?.1, SW?.1, SW?.1, SW?.1, SW?.1, SW?.1, SW?.1, SW?.1, SW?.1, SW?.1, SW?.1, SW?.1, SW?.1, SW?.1, U?.14 (V+), U?.14 (V+), U?.14 (V+), U?.14 (V+), U?.14 (V+), U?.14 (V+), U?.14 (V+), U?.14 (V+), U?.14 (V+), U?.14 (V+), U?.14 (V+), U?.14 (V+), U?.14 (V+), U?.14 (V+), U?.14 (V+), U?.14 (V+)
- net CS_CTRL: now also D?.1 (K), D?.1 (K), D?.1 (K), D?.1 (K), D?.1 (K), D?.1 (K), D?.1 (K), D?.1 (K), D?.1 (K), D?.1 (K), D?.1 (K), D?.1 (K), D?.1 (K), D?.1 (K), D?.1 (K), D?.1 (K), D?.1 (K)
- net DKA11: now also U?.2 (O/I), U?.2 (O/I), U?.2 (O/I), U?.2 (O/I), U?.2 (O/I), U?.2 (O/I), U?.2 (O/I), U?.2 (O/I), U?.2 (O/I), U?.2 (O/I), U?.2 (O/I), U?.2 (O/I), U?.2 (O/I), U?.2 (O/I), U?.2 (O/I), U?.2 (O/I)
- net GND: now also R?.2, R?.2, R?.2, R?.2, R?.2, R?.2, R?.2, R?.2, R?.2, R?.2, R?.2, R?.2, R?.2, R?.2, R?.2, U?.7 (V-), U?.7 (V-), U?.7 (V-), U?.7 (V-), U?.7 (V-), U?.7 (V-), U?.7 (V-), U?.7 (V-), U?.7 (V-), U?.7 (V-), U?.7 (V-), U?.7 (V-), U?.7 (V-), U?.7 (V-), U?.7 (V-)
- net KD2: now also U?.1 (I/O), U?.1 (I/O), U?.1 (I/O), U?.1 (I/O), U?.1 (I/O), U?.1 (I/O), U?.1 (I/O), U?.1 (I/O), U?.1 (I/O), U?.1 (I/O), U?.1 (I/O), U?.1 (I/O), U?.1 (I/O), U?.1 (I/O), U?.1 (I/O), U?.1 (I/O)
- new net: R?.1, U?.13 (ON) (x16)
- new net: D?.2 (A), D?.2 (A), R?.1, R?.2, SW?.2 (x3)
- new net: D?.2 (A), R?.1, R?.2, SW?.2 (x11)
- new net: D?.2 (A), D?.2 (A), D?.2 (A), D?.2 (A), SW?.2
- new net: R?.1, R?.2 (x2)
- new net: D?.1 (K), D?.1 (K) (x2)
- new net: R?.2, U?.7 (V-)
Other:
- moved on the sheet: C1, D?, R?, SW43, U1A
