File: zx_keyboard.sch (KiCad schematic (older format))
At the start: 141 parts, among them P1 CONN_02X08, SW1 KEY_1, SW10 KEY_0, SW11 KEY_Q, SW12 KEY_W, SW13 KEY_E, SW14 KEY_R, SW15 KEY_T, SW16 KEY_Y, SW17 KEY_U, SW18 KEY_I, SW19 KEY_O, SW2 KEY_2, SW20 KEY_P, SW21 KEY_A, SW22 KEY_S, SW23 KEY_D, SW24 KEY_F, SW25 KEY_G, SW26 KEY_H, SW27 KEY_J, SW28 KEY_K, SW29 KEY_L, SW3 KEY_3, SW30 KEY_EN, SW31 KEY_CS1, SW32 KEY_Z, SW33 KEY_X, SW34 KEY_C, SW35 KEY_V, SW36 KEY_B, SW37 KEY_N, SW38 KEY_M, SW39 KEY_SS1, SW4 KEY_4, SW40 KEY_SP, SW41 KEY_CS2, SW42 KEY_SS2, SW43 KEY_EDIT, SW44 KEY_CL, SW45 KEY_TV, SW46 KEY_IV, SW47 KEY_LEFT, SW48 KEY_DOWN, SW49 KEY_UP, SW5 KEY_5, SW50 KEY_RIGHT, SW51 KEY_GR, SW52 KEY_DEL, SW53 KEY_QUOT, SW54 KEY_SEM, SW55 KEY_BREAK, SW56 KEY_DOT, SW57 KEY_COMMA, SW58 KEY_EXT, SW6 KEY_6, SW7 KEY_7, SW8 KEY_8, SW9 KEY_9, U1 4066, U2 4066, U3 4066, U4 4066, U5 4066

Commit message: zx
Parts:
- removed D1, D2, D3, D4, D5, D6, D7, D8: BAT41, symbol D
- added Q1, Q2, Q3, Q4, Q5, Q6, Q7, Q8: BSS123, SOT-23, symbol BSS138
- added R40, R41, R42, R43, R44: 1K, symbol R
- added R45, R46, R47, R48, R49, R50, R51, R52: 100, symbol R
- added U6, U7: 74HC14, symbol 74HC14
Connections:
- net DKA11 is gone; now on net KA11: SW1.1, SW2.1, SW3.1, SW4.1, SW5.1, U1.2 (O/I), U1.2 (O/I), U1.2 (O/I), U1.2 (O/I), U2.2 (O/I)
- net DKA12 is gone; now on net KA12: SW10.1, SW6.1, SW7.1, SW8.1, SW9.1, U2.2 (O/I), U2.2 (O/I), U2.2 (O/I), U3.2 (O/I), U3.2 (O/I)
- net DKA13 is gone; now on net KA13: SW16.1, SW17.1, SW18.1, SW19.1, SW20.1, U3.2 (O/I), U3.2 (O/I)
- net DKA15 is gone; now on net KA15: SW36.1, SW37.1, SW38.1, SW39.1, SW40.1, SW42.1, U4.2 (O/I), U4.2 (O/I), U4.2 (O/I), U5.2 (O/I)
- net DKA8 is gone; now on net KA8: SW31.1, SW32.1, SW33.1, SW34.1, SW35.1, SW41.1, U5.2 (O/I)
- net +3V3: now also U6.14 (VCC), U6.14 (VCC), U6.14 (VCC), U6.14 (VCC), U6.14 (VCC), U6.14 (VCC), U7.14 (VCC), U7.14 (VCC)
- net GND: now also Q1.2 (S), Q2.2 (S), Q3.2 (S), Q4.2 (S), Q5.2 (S), Q6.2 (S), Q7.2 (S), Q8.2 (S), U6.7 (GND), U6.7 (GND), U6.7 (GND), U6.7 (GND), U6.7 (GND), U6.7 (GND), U7.7 (GND), U7.7 (GND)
- net KA10: now also SW11.1, SW12.1, SW13.1, SW14.1, SW15.1, Q3.3 (D); no longer P1.5 (P5)
- net KA11: now also Q4.3 (D); no longer P1.7 (P7)
- net KA12: now also Q5.3 (D); no longer P1.9 (P9)
- net KA13: now also Q6.3 (D); no longer P1.11 (P11)
- net KA14: now also SW26.1, SW27.1, SW28.1, SW29.1, SW30.1, Q7.3 (D); no longer P1.13 (P13)
- net KA15: now also Q8.3 (D); no longer P1.15 (P15)
- net KA8: now also Q1.3 (D); no longer P1.1 (P1)
- net KA9: now also SW21.1, SW22.1, SW23.1, SW24.1, SW25.1, Q2.3 (D); no longer P1.3 (P3)
- net KD0: now also R40.1; no longer P1.2 (P2)
- net KD1: now also R41.1; no longer P1.4 (P4)
- net KD2: now also R42.1; no longer P1.6 (P6)
- net KD3: now also R43.1; no longer P1.8 (P8)
- net KD4: now also R44.1; no longer P1.10 (P10)
- new net: R45.2, U6.2
- new net: R46.2, U6.4
- new net: R47.2, U6.6
- new net: R48.2, U6.8
- new net: R49.2, U6.10
- new net: R50.2, U6.12
- new net: R51.2, U7.2
- new net: R52.2, U7.4
- new net: Q1.1 (G), R45.1
- new net: Q2.1 (G), R46.1
- new net: Q3.1 (G), R47.1
- new net: Q4.1 (G), R48.1
- new net: Q5.1 (G), R49.1
- new net: Q6.1 (G), R50.1
- new net: Q7.1 (G), R51.1
- new net: Q8.1 (G), R52.1
- new net A10: P1.5 (P5), U6.5
- new net A11: P1.7 (P7), U6.9
- new net A12: P1.9 (P9), U6.11
- new net A13: P1.11 (P11), U6.13
- new net A14: P1.13 (P13), U7.1
- new net A15: P1.15 (P15), U7.3
- new net A8: P1.1 (P1), U6.1
- new net A9: P1.3 (P3), U6.3
- new net D0: P1.2 (P2), R40.2
- new net D1: P1.4 (P4), R41.2
- new net D2: P1.6 (P6), R42.2
- new net D3: P1.8 (P8), R43.2
- new net D4: P1.10 (P10), R44.2
Other:
- moved on the sheet: C1, D10, D11, D12, D13, D14, D15, D16, D17, D18, D19, D20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

Commit message: pcb
Parts:
- removed U1 (x3), U2 (x3), U3 (x3), U4 (x2), U5: 4066, TO_SOT_Packages_SMD:SOT-428, symbol 4066
- added unit 2 of U1
- added unit 3 of U1
- added unit 4 of U1
- added unit 2 of U2
- added unit 3 of U2
- added unit 4 of U2
- added unit 2 of U3
- added unit 3 of U3
- added unit 4 of U3
- added unit 2 of U4
- added unit 3 of U4
- added unit 2 of U5
- C1: footprint (none) -> Capacitors_Tantalum_SMD:TantalC_SizeC_EIA-6032_HandSoldering
- D1: renamed from D9; footprint (none) -> Diodes_ThroughHole:Diode_DO-35_SOD27_Horizontal_RM10
- D10: renamed from D18; footprint (none) -> Diodes_ThroughHole:Diode_DO-35_SOD27_Horizontal_RM10
- D11: renamed from D19; footprint (none) -> Diodes_ThroughHole:Diode_DO-35_SOD27_Horizontal_RM10
- D12: renamed from D20; footprint (none) -> Diodes_ThroughHole:Diode_DO-35_SOD27_Horizontal_RM10
- D13: renamed from D21; footprint (none) -> Diodes_ThroughHole:Diode_DO-35_SOD27_Horizontal_RM10
- D14: renamed from D22; footprint (none) -> Diodes_ThroughHole:Diode_DO-35_SOD27_Horizontal_RM10
- D15: renamed from D23; footprint (none) -> Diodes_ThroughHole:Diode_DO-35_SOD27_Horizontal_RM10
- D16: renamed from D24; footprint (none) -> Diodes_ThroughHole:Diode_DO-35_SOD27_Horizontal_RM10
- D17: renamed from D25; footprint (none) -> Diodes_ThroughHole:Diode_DO-35_SOD27_Horizontal_RM10
- D2: renamed from D10; footprint (none) -> Diodes_ThroughHole:Diode_DO-35_SOD27_Horizontal_RM10
- D3: renamed from D11; footprint (none) -> Diodes_ThroughHole:Diode_DO-35_SOD27_Horizontal_RM10
- D4: renamed from D12; footprint (none) -> Diodes_ThroughHole:Diode_DO-35_SOD27_Horizontal_RM10
- D5: renamed from D13; footprint (none) -> Diodes_ThroughHole:Diode_DO-35_SOD27_Horizontal_RM10
- D6: renamed from D14; footprint (none) -> Diodes_ThroughHole:Diode_DO-35_SOD27_Horizontal_RM10
- D7: renamed from D15; footprint (none) -> Diodes_ThroughHole:Diode_DO-35_SOD27_Horizontal_RM10
- D8: renamed from D16; footprint (none) -> Diodes_ThroughHole:Diode_DO-35_SOD27_Horizontal_RM10
- D9: renamed from D17; footprint (none) -> Diodes_ThroughHole:Diode_DO-35_SOD27_Horizontal_RM10
- P1: footprint (none) -> Pin_Headers:Pin_Header_Angled_2x08
- Q1, Q2, Q3, Q4, Q5, Q6, Q7, Q8: footprint SOT-23 -> TO_SOT_Packages_SMD:SOT-23
- R1, R10, R11, R12, R13, R14, R15, R16, R17, R18, R19, R2, R20, R21, R22, R23, R24, R25, R26, R27, R28, R29, R3, R30, R31, R32, R33, R34, R35, R36, R37, R38, R39, R4, R40, R41, R42, R43, R44, R45, R46, R47, R48, R49, R5, R50, R51, R52, R6, R7, R8, R9: footprint (none) -> Resistors_SMD:R_0805_HandSoldering
- U1, U2, U3, U4, U5: footprint TO_SOT_Packages_SMD:SOT-428 -> Housings_SSOP:TSSOP-14_4.4x5mm_Pitch0.65mm
- U6, U7: footprint (none) -> Housings_SOIC:SOIC-14_3.9x8.7mm_Pitch1.27mm
Connections:
- net +3V3: now also U1.14 (V+), U1.14 (V+), U1.14 (V+), U2.14 (V+), U2.14 (V+), U2.14 (V+), U3.14 (V+), U3.14 (V+), U3.14 (V+), U4.14 (V+), U4.14 (V+), U5.14 (V+)
- net GND: now also R39.2, U1.7 (V-), U1.7 (V-), U1.7 (V-), U2.7 (V-), U2.7 (V-), U2.7 (V-), U3.7 (V-), U3.7 (V-), U3.7 (V-), U4.7 (V-), U4.7 (V-), U5.7 (V-)
- net KA11: now also U1.10 (O/I), U1.3 (O/I), U1.9 (O/I)
- net KA12: now also U2.10 (O/I), U2.3 (O/I), U2.9 (O/I), U3.3 (O/I)
- net KA13: now also U3.10 (O/I), U3.9 (O/I)
- net KA15: now also U4.3 (O/I), U4.9 (O/I), U5.3 (O/I)
- net KD0: now also U3.4 (I/O), U3.8 (I/O)
- net KD1: now also U1.4 (I/O), U3.11 (I/O), U5.4 (I/O)
- net KD2: now also U1.8 (I/O), U2.11 (I/O), U4.4 (I/O)
- net KD3: now also U1.11 (I/O), U2.8 (I/O), U4.8 (I/O)
- net KD4: now also U2.4 (I/O)
- net at R8.1: now also U1.5 (ON)
- net at R10.1: now also U1.6 (ON)
- net at R16.1: now also U2.5 (ON)
- net at R18.1: now also U2.6 (ON)
- net at R20.1: now also U2.12 (ON)
- net at R26.1: now also U3.6 (ON)
- net at R28.1: now also U3.12 (ON)
- net at R12.1: now also U1.12 (ON)
- net at R32.1: now also U4.5 (ON)
- net at R24.1: now also U3.5 (ON)
- net at R34.1: now also U4.6 (ON)
- net at R38.1: now also U5.5 (ON)
