File: mainboard/zx_mainboard.kicad_pcb (KiCad board)
At the start: 2 copper layers, 93 parts, among them P1 CONN_02X17, P2 CONN_02X20, P3 CONN_02X20, P4 CONN_01X02, Q1 BSS123, Q2 BSS123, Q3 BSS123, Q4 BSS123, Q5 BSS123, Q6 BSS123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

Commit message: pcb
Parts:
- moved P1 225.8 mm to (62.2, 141.0), turned to 90 degrees
- moved P3 161.1 mm to (95.9, 90.2), turned to 270 degrees
- moved P2 103.1 mm to (131.4, 94.0), turned to 180 degrees
- moved D1 87.7 mm to (174.6, 148.7)
- moved D11 87.7 mm to (175.1, 141.7)
- moved D12 87.7 mm to (175.1, 156.7)
- moved D14 87.7 mm to (156.6, 167.2)
- moved D15 87.7 mm to (153.6, 159.7)
- moved D16 87.7 mm to (154.6, 151.7)
- moved D17 87.7 mm to (157.6, 144.2)
- moved D4 87.7 mm to (172.6, 171.2)
- moved D6 87.7 mm to (174.1, 145.7)
- moved D7 87.7 mm to (173.1, 177.7)
- moved D8 87.7 mm to (176.1, 163.2)
- moved U3 87.7 mm to (199.1, 167.7)
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Other:
- board outline added: 130.2 x 130.2 mm

Commit message: mainboard pcb
Parts:
- D1, D10, D11, D12, D13, D14, D15, D16, D17, D2, D3, D4, D5, D6, D7, D8, D9: moved to B.Cu
- moved C2 251.7 mm to (30.5, 93.3), turned to 90 degrees
- moved R8 220.5 mm to (22.9, 110.5), turned to 180 degrees
- moved R9 220.2 mm to (22.9, 108.0)
- moved R46 219.3 mm to (38.7, 122.6)
- moved R10 219.2 mm to (22.9, 113.0), turned to 180 degrees
- moved R2 211.7 mm to (28.6, 134.6), turned to 90 degrees
- moved R47 210.0 mm to (51.4, 122.6)
- moved R3 196.4 mm to (33.0, 134.6), turned to 270 degrees
- moved R16 195.4 mm to (48.3, 110.5), turned to 180 degrees
- moved R7 194.0 mm to (38.1, 108.0), turned to 180 degrees
- moved Q1 192.2 mm to (21.0, 123.8), turned to 180 degrees
- moved Q4 192.1 mm to (59.1, 123.8), turned to 180 degrees
- moved R11 191.2 mm to (22.9, 115.6)
- moved R45 189.1 mm to (26.0, 122.6)
- moved Q2 189.0 mm to (33.7, 123.8), turned to 180 degrees
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Other:
- outline, holes or cut-outs redrawn
- net class Default: trace_width 0.25 -> 0.4; via_dia 0.6 -> 1; via_drill 0.4 -> 0.6

Commit message: pcb
Parts:
- D1, D10, D11, D12, D13, D14, D15, D16, D17, D2, D3, D4, D5, D6, D7, D8, D9: moved to F.Cu
- moved C2 103.1 mm to (133.3, 99.7), turned to 0 degrees
- moved D11 87.1 mm to (175.9, 99.1), turned to 0 degrees
- moved D12 80.8 mm to (175.9, 102.9), turned to 0 degrees
- moved D14 75.0 mm to (175.9, 106.7), turned to 0 degrees
- moved D15 69.6 mm to (175.9, 110.5), turned to 0 degrees
- moved D17 62.4 mm to (175.9, 114.3), turned to 0 degrees
- moved R44 61.7 mm to (80.0, 106.0), turned to 180 degrees
- moved R41 56.8 mm to (149.9, 110.5), turned to 0 degrees
- moved D6 56.0 mm to (184.2, 127.6), turned to 270 degrees
- moved R40 49.7 mm to (132.1, 102.9), turned to 180 degrees
- moved C1 47.0 mm to (154.9, 99.7), turned to 180 degrees
- moved R43 40.9 mm to (139.7, 113.0)
- moved U6 35.3 mm to (174.0, 55.9), turned to 90 degrees
- moved U7 34.5 mm to (174.0, 73.0), turned to 90 degrees
- moved R42 29.2 mm to (132.1, 106.7)
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Connections:
- C2 pad 1: +3V3 -> +5V
- P2 pad 2: /VCC_5V -> +5V
- P2 pad 4: /VCC_5V -> +5V
- P3 pad 2: /VCC_5V -> +5V
- P3 pad 4: /VCC_5V -> +5V
Routing:
- net +3V3: track 0.00 -> 221.9 mm
- net GND: track 0.00 -> 107.5 mm, vias 0 -> 30
- net /GPIO17: track 0.00 -> 102.2 mm
- net /GPIO8: track 0.00 -> 77.9 mm, vias 0 -> 2
- net /GPIO7: track 0.00 -> 72.9 mm, vias 0 -> 2
- net /CS_CTRL: track 0.00 -> 68.1 mm
- net /GPIO4: track 0.00 -> 66.5 mm, vias 0 -> 2
- net /SS_CTRL: track 0.00 -> 59.0 mm, vias 0 -> 2
- net Net-(R52-Pad2): track 0.00 -> 52.5 mm, vias 0 -> 4
- net +5V: track 0.00 -> 51.0 mm
- net /GPIO9: track 0.00 -> 28.7 mm, vias 0 -> 1
- net /GPIO6: track 0.00 -> 25.9 mm, vias 0 -> 1
- net /GPIO11: track 0.00 -> 23.2 mm, vias 0 -> 2
- net /GPIO5: track 0.00 -> 18.6 mm, vias 0 -> 2
- net /GPIO10: track 0.00 -> 16.6 mm, vias 0 -> 1
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- added copper zone on B.Cu, net GND
Other:
- board size 130.2 x 130.2 mm -> 149.9 x 130.2 mm

Commit message: pcb
Parts:
- added P5: CONN_01X02, Connectors_Phoenix:PhoenixContact_MCV-G_02x5.08mm_Vertical, F.Cu at (184.2, 92.7)
- D10, D11, D12, D13, D14, D15, D16, D17, D9: moved to B.Cu
- moved D11 70.7 mm to (108.0, 118.7), turned to 180 degrees
- moved R55 62.6 mm to (106.7, 141.6), turned to 0 degrees
- moved D12 52.4 mm to (126.4, 120.0), turned to 180 degrees
- moved D14 48.4 mm to (128.9, 118.1), turned to 180 degrees
- moved D15 44.7 mm to (131.4, 115.6), turned to 180 degrees
- moved D17 44.6 mm to (131.4, 118.1), turned to 270 degrees
- moved D6 26.0 mm to (158.1, 127.6)
- moved D5 19.0 mm to (161.3, 127.6)
- moved D1 16.5 mm to (174.0, 127.6)
- moved D9 12.5 mm to (153.7, 132.7), turned to 180 degrees
- moved D4 12.1 mm to (164.5, 127.6)
- moved D16 11.7 mm to (153.7, 130.2), turned to 180 degrees
- moved D13 9.86 mm to (143.5, 118.1), turned to 90 degrees
- moved D8 9.52 mm to (151.8, 127.6)
- moved D10 8.52 mm to (153.7, 135.3), turned to 180 degrees
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Routing:
- net /KEDIT: track 2.54 -> 76.2 mm
- net /KCL: track 2.54 -> 68.6 mm
- net /KTV: track 2.54 -> 63.5 mm
- net /KIV: track 2.54 -> 61.6 mm
- net /KLEFT: track 2.54 -> 54.6 mm
- net /KDOWN: track 2.54 -> 45.7 mm
- net +5V: track 51.0 -> 93.5 mm
- net /KGR: track 2.66 -> 44.1 mm
- net /KDEL: track 2.54 -> 38.9 mm
- net /KUP: track 2.54 -> 38.7 mm
- net /KRIGHT: track 2.54 -> 32.0 mm
- net /KD4: track 0.00 -> 24.1 mm
- net /KEXT: track 0.00 -> 24.0 mm
- net /KD0: track 6.71 -> 28.3 mm
- net /CS_CTRL: track 68.1 -> 88.6 mm
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Other:
- net class Default: via_dia 1 -> 1.5
- net class power added: clearance 0.4, trace_width 1, via_dia 1.5, via_drill 0.6

Commit message: pcb
Parts:
- D10, D13, D16, D9: moved to F.Cu
- moved R45 162.6 mm to (214.0, 122.6)
- moved Q1 159.4 mm to (205.7, 120.0)
- moved R46 141.6 mm to (203.8, 99.7)
- moved Q2 141.1 mm to (197.5, 96.5)
- moved R47 137.5 mm to (213.4, 106.0)
- moved Q3 134.1 mm to (205.1, 109.9)
- moved R48 131.7 mm to (212.1, 74.3)
- moved Q4 130.1 mm to (205.7, 76.8)
- moved R49 99.5 mm to (207.0, 61.0)
- moved Q5 98.1 mm to (200.7, 62.9)
- moved R50 68.5 mm to (209.6, 131.4)
- moved R51 67.1 mm to (210.8, 86.4)
- moved Q6 65.7 mm to (201.9, 129.5)
- moved Q7 64.6 mm to (203.2, 88.3)
- moved Q8 36.0 mm to (170.8, 88.9)
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Routing:
- net /KIV: track 61.6 -> 208.2 mm, vias 0 -> 4
- net /KCL: track 68.6 -> 202.0 mm, vias 0 -> 7
- net /KTV: track 63.5 -> 191.2 mm, vias 0 -> 1
- net /KD0: track 28.3 -> 146.9 mm, vias 0 -> 7
- net /KEDIT: track 76.2 -> 178.3 mm, vias 0 -> 1
- net /KUP: track 38.7 -> 138.6 mm, vias 0 -> 6
- net /KD1: track 6.71 -> 104.9 mm, vias 0 -> 2
- net /GPIO19: track 0.00 -> 78.1 mm, vias 0 -> 1
- net /GPIO26: track 0.00 -> 70.5 mm
- net GND: track 110.7 -> 172.0 mm, vias 30 -> 26
- net /GPIO21: track 0.00 -> 54.0 mm
- net /GPIO20: track 0.00 -> 50.2 mm
- net /KD2: track 20.3 -> 69.9 mm, vias 0 -> 2
- net /KD3: track 0.00 -> 49.5 mm, vias 0 -> 2
- net /KA11: track 7.74 -> 53.8 mm, vias 0 -> 4
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Other:
- outline, holes or cut-outs redrawn

Commit message: pcb
Parts:
- moved R50 99.8 mm to (169.5, 40.0), turned to 270 degrees
- moved Q6 99.0 mm to (170.8, 35.6), turned to 0 degrees
- moved R45 78.6 mm to (171.4, 56.5), turned to 90 degrees
- moved Q1 68.4 mm to (170.2, 61.6), turned to 270 degrees
- moved R47 61.7 mm to (176.5, 56.5), turned to 90 degrees
- moved Q3 54.8 mm to (179.1, 61.6), turned to 270 degrees
- moved R46 52.5 mm to (174.0, 56.5), turned to 90 degrees
- moved Q4 48.8 mm to (179.7, 35.6), turned to 0 degrees
- moved R48 48.0 mm to (178.4, 40.0), turned to 270 degrees
- moved Q2 41.7 mm to (174.6, 61.6), turned to 270 degrees
- moved R51 39.9 mm to (171.4, 80.0), turned to 90 degrees
- moved R49 39.1 mm to (174.0, 40.0), turned to 270 degrees
- moved Q5 37.3 mm to (175.3, 35.6), turned to 0 degrees
- moved Q7 33.2 mm to (170.2, 85.1)
- moved P5 27.3 mm to (184.2, 120.0)
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Routing:
- net /GPIO17: track 102.2 -> 0.00 mm
- net /KA8: track 5.71 -> 105.2 mm, vias 0 -> 2
- net /KA13: track 0.65 -> 91.7 mm
- net /KA12: track 14.6 -> 96.8 mm
- net /KA11: track 53.8 -> 127.7 mm
- net GND: track 172.0 -> 102.4 mm, vias 26 -> 29
- net /KA9: track 0.00 -> 45.2 mm
- net /KA10: track 10.2 -> 52.3 mm
- net /KA15: track 47.9 -> 82.1 mm
- net /GPIO4: track 69.1 -> 42.5 mm, vias 2 -> 4
- net /KA14: track 17.8 -> 40.3 mm
- net +5V: track 93.5 -> 113.2 mm
- net /GPIO9: track 28.7 -> 38.2 mm, vias 1 -> 6
- net Net-(R52-Pad2): track 11.5 -> 2.94 mm, vias 2 -> 0
- net Net-(R50-Pad2): track 0.00 -> 7.69 mm
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
Commit message: pcb
Parts:
- moved D17 6.35 mm to (137.8, 118.1)
- moved R4 3.24 mm to (83.2, 120.0)
- moved R16 2.29 mm to (71.8, 108.6)
- moved R17 2.29 mm to (71.8, 106.0)
- moved D11 1.27 mm to (106.7, 118.7)
- moved R24 1.27 mm to (97.8, 110.5)
- moved R26 1.27 mm to (97.8, 113.0)
- moved R27 1.27 mm to (97.8, 115.6)
- moved R14 0.63 mm to (89.5, 110.5)
- moved R15 0.63 mm to (89.5, 108.0)
- moved R20 0.63 mm to (89.5, 113.0)
- moved R21 0.63 mm to (89.5, 115.6)
Routing:
- net /KDOWN: track 59.1 -> 192.6 mm, vias 0 -> 4
- net /GPIO16: track 0.00 -> 130.3 mm, vias 0 -> 8
- net /KLEFT: track 67.3 -> 178.4 mm, vias 0 -> 5
- net /KA8: track 105.2 -> 204.8 mm, vias 2 -> 3
- net /KD3: track 49.5 -> 147.3 mm, vias 2 -> 7
- net /KD1: track 104.9 -> 186.4 mm, vias 2 -> 4
- net /KD2: track 69.9 -> 151.0 mm, vias 2 -> 6
- net /KA12: track 96.8 -> 171.3 mm, vias 0 -> 4
- net /KD0: track 146.9 -> 218.7 mm, vias 7 -> 10
- net /GPIO12: track 0.00 -> 68.4 mm, vias 0 -> 4
- net /KRIGHT: track 40.7 -> 106.0 mm, vias 0 -> 4
- net /GPIO2: track 17.8 -> 76.2 mm, vias 0 -> 2
- net /KDEL: track 38.9 -> 83.2 mm, vias 0 -> 3
- net /GPIO14: track 0.00 -> 39.5 mm, vias 0 -> 4
- net /KA11: track 127.7 -> 165.3 mm, vias 4 -> 5
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
Commit message: pcb
Parts:
- removed R55: 0R, Resistors_SMD:R_0805_HandSoldering
- moved P5 22.9 mm to (171.4, 101.0)
Connections:
- P1 pad 15: Net-(P1-Pad15) -> +3V3
- P1 pad 16: Net-(P1-Pad16) -> +3V3
- P1 pad 17: /KCOMM -> +3V3
Routing:
- net +3V3: track 267.4 -> 340.4 mm
- net +5V: track 147.5 -> 110.7 mm
- net /GPIO2: track 76.2 -> 68.0 mm, vias 2 -> 1
- net /KA15: track 117.6 -> 109.5 mm
- net /KCOMM: track 3.21 -> 0.00 mm
- net /KA8: track 204.8 -> 207.4 mm
