File: mainboard/zx_mainboard.kicad_pcb (KiCad board)
At the start: 2 copper layers, 149.9 x 130.2 mm, 93 parts, among them P1 CONN_02X17, P2 CONN_02X20, P3 CONN_02X20, P4 CONN_01X02, P5 CONN_01X02, Q1 BSS123, Q2 BSS123, Q3 BSS123, Q4 BSS123, Q5 BSS123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

Commit message: pcb
Parts:
- moved D12 3.81 mm to (122.6, 120.0)
- moved D13 3.24 mm to (144.1, 121.3)
- moved D14 1.91 mm to (130.8, 118.1)
Routing:
- net /GPIO17: track 0.00 -> 96.5 mm, vias 0 -> 5
- net /KA13: track 91.7 -> 188.1 mm, vias 0 -> 4
- net /KA12: track 171.3 -> 259.2 mm, vias 4 -> 6
- net /GPIO13: track 0.11 -> 83.6 mm, vias 0 -> 5
- net /KGR: track 42.3 -> 104.3 mm, vias 0 -> 2
- net /KA11: track 165.3 -> 223.7 mm, vias 5 -> 6
- net /GPIO15: track 0.00 -> 49.3 mm, vias 0 -> 4
- net /KBREAK: track 5.01 -> 54.1 mm, vias 0 -> 4
- net /KA9: track 45.2 -> 93.5 mm, vias 0 -> 1
- net /KA10: track 51.7 -> 96.2 mm, vias 0 -> 1
- net /KA8: track 207.4 -> 233.0 mm, vias 3 -> 4
- net /KA14: track 40.3 -> 65.0 mm, vias 0 -> 1
- net /KCOMMA: track 5.30 -> 28.1 mm
- net /KSEM: track 7.21 -> 27.9 mm, vias 0 -> 1
- net /KDOT: track 13.3 -> 32.9 mm
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- added copper zone on F.Cu, net +3V3

Commit message: pcb
Routing:
- net /KA15: track 113.6 -> 156.2 mm
- net +3V3: track 340.4 -> 345.0 mm
- net /KA8: track 233.0 -> 230.3 mm
- net /GPIO16: track 136.4 -> 133.8 mm
- net /KDEL: track 89.5 -> 87.0 mm, vias 3 -> 4
- net /KGR: vias 2 -> 3
- added copper zone on B.Cu, net +3V3
- removed copper zone on F.Cu, net +3V3

Commit message: pcb
Parts:
- moved R29 1.90 mm to (114.3, 113.7)
- moved R22 1.42 mm to (115.6, 109.9)
- moved R23 1.27 mm to (115.6, 108.0)
- moved R28 1.27 mm to (114.3, 111.8)
- moved R40 0.90 mm to (131.4, 103.5)
- moved R30 0.64 mm to (140.3, 110.5)
- moved R31 0.64 mm to (140.3, 108.0)
- moved R43 0.64 mm to (140.3, 113.0)
- moved R42 0.63 mm to (132.1, 107.3)
Routing:
- net /GPIO19: track 78.1 -> 176.8 mm, vias 1 -> 4
- net /GPIO20: track 50.2 -> 144.8 mm, vias 0 -> 4
- net /GPIO26: track 70.5 -> 160.5 mm, vias 0 -> 4
- net /GPIO21: track 54.0 -> 131.6 mm, vias 0 -> 4
- net +3V3: track 345.0 -> 416.0 mm, vias 0 -> 1
- net /GPIO3: track 0.00 -> 68.5 mm, vias 0 -> 1
- net /GPIO18: track 22.9 -> 67.3 mm, vias 1 -> 4
- net /KD1: track 187.1 -> 226.4 mm, vias 4 -> 7
- net /KA8: track 230.3 -> 207.0 mm
- net /GPIO8: track 82.7 -> 67.4 mm, vias 2 -> 3
- net /GPIO7: track 77.2 -> 64.5 mm, vias 2 -> 3
- net /KLEFT: track 188.6 -> 178.0 mm
- net /KA13: track 188.1 -> 180.2 mm
- net /GPIO14: track 39.5 -> 44.8 mm, vias 4 -> 5
- net /GPIO15: track 49.3 -> 53.9 mm, vias 4 -> 5
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- removed copper zone on B.Cu, net +3V3
Other:
- outline, holes or cut-outs redrawn

Commit message: pcb
Routing:
- net /KA9: track 93.5 -> 196.4 mm, vias 1 -> 4
- net /KA12: track 257.5 -> 349.4 mm
- net /KA11: track 223.7 -> 313.0 mm, vias 6 -> 8
- net /KA13: track 180.2 -> 254.4 mm, vias 4 -> 5
- net /KA15: track 152.8 -> 218.2 mm, vias 3 -> 5
- net /CS_CTRL: track 114.8 -> 125.1 mm, vias 0 -> 3
- net /KCL: track 200.1 -> 189.8 mm, vias 5 -> 3
- net /KA10: track 96.2 -> 89.2 mm
- net /KD4: track 73.2 -> 79.6 mm
- net /KRIGHT: track 106.9 -> 112.8 mm
- net /KD1: track 226.4 -> 221.1 mm
- net /KA8: track 207.0 -> 202.1 mm, vias 4 -> 2
- net /KD2: track 151.1 -> 155.7 mm, vias 8 -> 6
- net /KLEFT: track 178.0 -> 174.7 mm, vias 5 -> 3
- net +5V: track 106.4 -> 104.1 mm
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
Commit message: pcb
Parts:
- moved D11 0.64 mm to (106.7, 118.1)
- moved D14 0.63 mm to (130.2, 118.1)
Routing:
- net /KA10: track 89.2 -> 233.4 mm, vias 1 -> 2
- net /KA14: track 65.0 -> 103.8 mm
- net /KEXT: track 27.8 -> 47.2 mm, vias 0 -> 1
- net /KA15: track 218.2 -> 236.3 mm
- net /KA12: track 349.4 -> 340.5 mm
- net /KRIGHT: track 112.8 -> 104.0 mm
- net /SS_CTRL: track 67.0 -> 70.9 mm
- net /KA13: track 254.4 -> 258.3 mm
- net /KD3: track 148.1 -> 151.8 mm
- net /KLEFT: track 174.7 -> 177.5 mm
- net /KQUOT: track 39.8 -> 42.5 mm
- net /KA9: track 196.4 -> 198.3 mm, vias 4 -> 3
- net /KBREAK: track 55.3 -> 57.1 mm, vias 4 -> 2
- net /KDEL: track 87.8 -> 89.4 mm
- net /KCOMMA: track 28.1 -> 29.7 mm
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
Commit message: pcb
Parts:
- moved R11 1.42 mm to (48.3, 116.2)
- moved R1 1.27 mm to (54.0, 106.0)
- moved R10 0.90 mm to (47.6, 113.7)
- moved R8 0.63 mm to (47.6, 110.5)
Routing:
- net /KA14: track 103.8 -> 187.3 mm, vias 1 -> 2
- net /GPIO16: track 131.9 -> 199.1 mm
- net /GPIO26: track 160.5 -> 214.5 mm
- net /GPIO12: track 75.5 -> 123.1 mm
- net /KA15: track 236.3 -> 190.9 mm
- net /GPIO20: track 144.8 -> 184.6 mm
- net /KA10: track 233.4 -> 197.0 mm
- net /GPIO19: track 176.8 -> 212.1 mm
- net /GPIO18: track 67.3 -> 99.7 mm
- net /KA11: track 312.0 -> 283.0 mm
- net /KA12: track 340.5 -> 316.0 mm
- net /GPIO3: track 68.5 -> 86.9 mm
- net /KD0: track 223.9 -> 241.2 mm
- net /KGR: track 105.1 -> 88.4 mm
- net /GPIO21: track 131.6 -> 148.3 mm
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Other:
- outline, holes or cut-outs redrawn

Commit message: pcb
Parts:
- moved R54 5.08 mm to (161.3, 37.5)
- moved D5 4.45 mm to (169.5, 127.6)
- moved D1 4.44 mm to (182.2, 127.6)
- moved D2 4.44 mm to (179.1, 127.6)
- moved D3 4.44 mm to (175.9, 127.6)
- moved D4 4.44 mm to (172.7, 127.6)
- moved D6 4.44 mm to (166.4, 127.6)
- moved D7 4.44 mm to (163.2, 127.6)
- moved D8 4.44 mm to (160.0, 127.6)
- moved C2 4.02 mm to (134.6, 95.9)
- moved R44 1.42 mm to (79.4, 103.5)
- moved R5 1.42 mm to (79.4, 106.0)
Routing:
- net /GPIO16: track 199.1 -> 152.5 mm
- net +3V3: track 415.5 -> 369.2 mm
- net /GPIO12: track 123.1 -> 83.7 mm
- net /GPIO17: track 90.9 -> 52.2 mm, vias 5 -> 2
- net /GPIO20: track 184.6 -> 164.9 mm
- net /GPIO4: track 42.5 -> 61.8 mm, vias 4 -> 2
- net /CS_CTRL: track 125.1 -> 111.1 mm
- net /KIV: track 206.6 -> 194.0 mm
- net /KA10: track 197.0 -> 184.4 mm
- net /KLEFT: track 177.5 -> 165.2 mm
- net /KDOWN: track 190.0 -> 178.4 mm
- net /GPIO19: track 212.1 -> 201.1 mm
- net /GPIO6: track 34.4 -> 24.9 mm, vias 2 -> 1
- net /KD1: track 214.1 -> 204.8 mm
- net /GPIO26: track 214.5 -> 205.6 mm
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Other:
- board size 149.9 x 130.2 mm -> 146.1 x 123.8 mm
- net class 3.3v added: clearance 0.2, trace_width 0.45, via_dia 1.5, via_drill 0.6
- board text added: "ZX mainboard v0.1"

Commit message: pcb
Parts:
- U1, U2, U3, U4, U5: footprint Housings_SSOP:TSSOP-14_4.4x5mm_Pitch0.65mm -> Housings_SOIC:SOIC-14_3.9x8.7mm_Pitch1.27mm
- moved R42 3.24 mm to (131.4, 104.1)
- moved R37 3.18 mm to (165.1, 110.5)
- moved R22 3.17 mm to (113.7, 107.3)
- moved R30 3.17 mm to (140.3, 107.3)
- moved R31 3.17 mm to (140.3, 104.8)
- moved R25 2.84 mm to (97.8, 105.4)
- moved R33 2.69 mm to (121.3, 106.0), turned to 180 degrees
- moved R36 2.54 mm to (165.1, 108.0)
- moved R1 2.29 mm to (55.2, 104.1)
- moved R5 2.29 mm to (78.1, 104.1), turned to 90 degrees
- moved R23 2.01 mm to (117.5, 107.3), turned to 90 degrees
- moved R28 2.01 mm to (113.7, 109.9)
- moved R2 1.91 mm to (55.2, 101.6)
- moved R29 1.91 mm to (114.3, 111.8)
- moved R40 1.91 mm to (131.4, 101.6)
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Routing:
- net /KD1: track 204.8 -> 150.6 mm, vias 7 -> 4
- net +3V3: track 369.2 -> 354.4 mm
- net /KD0: track 233.4 -> 220.5 mm, vias 11 -> 7
- net /KD3: track 150.1 -> 140.0 mm
- net /KSEM: track 27.2 -> 35.9 mm
- net /GPIO12: track 83.7 -> 75.4 mm
- net /KDEL: track 88.7 -> 82.0 mm
- net /GPIO14: track 48.8 -> 44.1 mm
- net /KD4: track 80.2 -> 84.7 mm, vias 3 -> 1
- net /KA15: track 186.7 -> 182.9 mm
- net GND: track 97.1 -> 93.5 mm, vias 29 -> 28
- net /KGR: track 88.4 -> 91.2 mm
- net /CS_CTRL: track 111.1 -> 108.3 mm
- net /KA8: track 188.3 -> 191.0 mm
- net /KCL: track 180.3 -> 182.8 mm
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