File: mainboard/zx_mainboard.kicad_pcb (KiCad board)
At the start: 2 copper layers, 146.1 x 123.8 mm, 93 parts, among them P1 CONN_02X17, P2 CONN_02X20, P3 CONN_02X20, P4 CONN_01X02, P5 CONN_01X02, Q1 BSS123, Q2 BSS123, Q3 BSS123, Q4 BSS123, Q5 BSS123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

Commit message: pcb
Parts:
- moved R42 6.76 mm to (125.5, 107.3), turned to 270 degrees
- moved R30 3.17 mm to (140.3, 110.5)
- moved R31 3.17 mm to (140.3, 108.0)
- moved R24 2.01 mm to (99.7, 111.1)
- moved R27 2.01 mm to (99.7, 114.9)
- moved R26 1.90 mm to (99.7, 113.0)
- moved R25 1.65 mm to (98.4, 103.9), turned to 180 degrees
- moved R33 1.42 mm to (121.9, 107.3), turned to 90 degrees
- moved R28 1.27 mm to (113.7, 108.6)
- moved D11 1.27 mm to (108.0, 118.1)
- moved R22 1.27 mm to (113.7, 106.0)
- moved R29 1.27 mm to (114.3, 113.0)
- moved R43 0.90 mm to (141.0, 113.0)
- moved R23 0.64 mm to (118.1, 107.3)
- moved R32 0.64 mm to (123.2, 111.1)
Routing:
- net /KD1: track 150.6 -> 182.4 mm, vias 4 -> 3
- net GND: track 93.5 -> 105.7 mm, vias 28 -> 27
- net /KD2: track 158.9 -> 150.0 mm
- net /KA15: track 182.9 -> 191.1 mm, vias 5 -> 7
- net /SS_CTRL: track 70.9 -> 65.4 mm
- net /KD0: track 220.5 -> 226.0 mm, vias 7 -> 8
- net /GPIO12: track 75.4 -> 71.4 mm
- net /GPIO14: track 44.1 -> 48.0 mm
- net +3V3: track 354.4 -> 351.1 mm
- net /KA13: track 252.2 -> 249.0 mm
- net /KDOT: track 33.7 -> 30.5 mm
- net /KBREAK: track 59.2 -> 56.7 mm
- net Net-(R30-Pad1): track 4.21 -> 6.64 mm
- net /KGR: track 91.2 -> 93.5 mm
- net /KQUOT: track 41.0 -> 38.8 mm
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Other:
- board text added: "ZX Mainboard v0.1"
- board text removed: "ZX mainboard v0.1"

Commit message: pcb
Parts:
- moved C1 5.12 mm to (160.0, 100.3), turned to 0 degrees
- moved P5 1.42 mm to (170.8, 99.7)
- moved R41 1.27 mm to (149.9, 109.2)
- moved D14 0.64 mm to (129.5, 118.1)
- moved R38 0.63 mm to (150.5, 113.0)
- moved R39 0.63 mm to (150.5, 115.6)
- moved R43 0.63 mm to (140.3, 113.0)
- moved U4 0.63 mm to (132.7, 109.9)
Routing:
- net /GPIO13: track 82.3 -> 96.3 mm
- net /KA15: track 191.1 -> 179.2 mm, vias 7 -> 5
- net /GPIO3: track 88.1 -> 78.2 mm
- net GND: track 105.7 -> 98.2 mm
- net /GPIO15: track 51.6 -> 44.2 mm
- net /KD0: track 226.0 -> 231.4 mm
- net /GPIO12: track 71.4 -> 67.8 mm
- net /SS_CTRL: track 65.4 -> 62.0 mm
- net /GPIO2: track 76.3 -> 79.3 mm
- net /GPIO14: track 48.0 -> 51.0 mm
- net /KD1: track 182.4 -> 184.7 mm
- net /KBREAK: track 56.7 -> 58.8 mm
- net /KD3: track 138.9 -> 136.9 mm
- net +3V3: track 351.1 -> 349.5 mm
- net Net-(R34-Pad1): track 5.17 -> 5.80 mm
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Other:
- outline, holes or cut-outs redrawn
