File: mainboard/zx_mainboard.sch (KiCad schematic (older format))
At the start: 144 parts, among them P1 CONN_02X08, Q1 BSS123, Q2 BSS123, Q3 BSS123, Q4 BSS123, Q5 BSS123, Q6 BSS123, Q7 BSS123, Q8 BSS123, SW1 KEY_1, SW10 KEY_0, SW11 KEY_Q, SW12 KEY_W, SW13 KEY_E, SW14 KEY_R, SW15 KEY_T, SW16 KEY_Y, SW17 KEY_U, SW18 KEY_I, SW19 KEY_O, SW2 KEY_2, SW20 KEY_P, SW21 KEY_A, SW22 KEY_S, SW23 KEY_D, SW24 KEY_F, SW25 KEY_G, SW26 KEY_H, SW27 KEY_J, SW28 KEY_K, SW29 KEY_L, SW3 KEY_3, SW30 KEY_EN, SW31 KEY_CS1, SW32 KEY_Z, SW33 KEY_X, SW34 KEY_C, SW35 KEY_V, SW36 KEY_B, SW37 KEY_N, SW38 KEY_M, SW39 KEY_SS1, SW4 KEY_4, SW40 KEY_SP, SW41 KEY_CS2, SW42 KEY_SS2, SW43 KEY_EDIT, SW44 KEY_CL, SW45 KEY_TV, SW46 KEY_IV, SW47 KEY_LEFT, SW48 KEY_DOWN, SW49 KEY_UP, SW5 KEY_5, SW50 KEY_RIGHT, SW51 KEY_GR, SW52 KEY_DEL, SW53 KEY_QUOT, SW54 KEY_SEM, SW55 KEY_BREAK, SW56 KEY_DOT, SW57 KEY_COMMA, SW58 KEY_EXT, SW6 KEY_6, SW7 KEY_7, SW8 KEY_8, SW9 KEY_9, U1 4066, U2 4066, U3 4066, U4 4066, U5 4066, U6 74HC14, U7 74HC14

Commit message: mainboard schematics & pcb
Parts:
- removed P1: CONN_02X08, Pin_Headers:Pin_Header_Angled_2x08, symbol CONN_02X08
- removed SW1: KEY_1, Buttons_Switches_Keyboard:SW_Cherry_MX1A_1.00u_PCB, symbol SW_PUSH
- removed SW10: KEY_0, Buttons_Switches_Keyboard:SW_Cherry_MX1A_1.00u_PCB, symbol SW_PUSH
- removed SW11: KEY_Q, Buttons_Switches_Keyboard:SW_Cherry_MX1A_1.00u_PCB, symbol SW_PUSH
- removed SW12: KEY_W, Buttons_Switches_Keyboard:SW_Cherry_MX1A_1.00u_PCB, symbol SW_PUSH
- removed SW13: KEY_E, Buttons_Switches_Keyboard:SW_Cherry_MX1A_1.00u_PCB, symbol SW_PUSH
- removed SW14: KEY_R, Buttons_Switches_Keyboard:SW_Cherry_MX1A_1.00u_PCB, symbol SW_PUSH
- removed SW15: KEY_T, Buttons_Switches_Keyboard:SW_Cherry_MX1A_1.00u_PCB, symbol SW_PUSH
- removed SW16: KEY_Y, Buttons_Switches_Keyboard:SW_Cherry_MX1A_1.00u_PCB, symbol SW_PUSH
- removed SW17: KEY_U, Buttons_Switches_Keyboard:SW_Cherry_MX1A_1.00u_PCB, symbol SW_PUSH
- removed SW18: KEY_I, Buttons_Switches_Keyboard:SW_Cherry_MX1A_1.00u_PCB, symbol SW_PUSH
- removed SW19: KEY_O, Buttons_Switches_Keyboard:SW_Cherry_MX1A_1.00u_PCB, symbol SW_PUSH
- removed SW2: KEY_2, Buttons_Switches_Keyboard:SW_Cherry_MX1A_1.00u_PCB, symbol SW_PUSH
- removed SW20: KEY_P, Buttons_Switches_Keyboard:SW_Cherry_MX1A_1.00u_PCB, symbol SW_PUSH
- removed SW21: KEY_A, Buttons_Switches_Keyboard:SW_Cherry_MX1A_1.00u_PCB, symbol SW_PUSH
- removed SW22: KEY_S, Buttons_Switches_Keyboard:SW_Cherry_MX1A_1.00u_PCB, symbol SW_PUSH
- removed SW23: KEY_D, Buttons_Switches_Keyboard:SW_Cherry_MX1A_1.00u_PCB, symbol SW_PUSH
- removed SW24: KEY_F, Buttons_Switches_Keyboard:SW_Cherry_MX1A_1.00u_PCB, symbol SW_PUSH
- removed SW25: KEY_G, Buttons_Switches_Keyboard:SW_Cherry_MX1A_1.00u_PCB, symbol SW_PUSH
- removed SW26: KEY_H, Buttons_Switches_Keyboard:SW_Cherry_MX1A_1.00u_PCB, symbol SW_PUSH
- removed SW27: KEY_J, Buttons_Switches_Keyboard:SW_Cherry_MX1A_1.00u_PCB, symbol SW_PUSH
- removed SW28: KEY_K, Buttons_Switches_Keyboard:SW_Cherry_MX1A_1.00u_PCB, symbol SW_PUSH
- removed SW29: KEY_L, Buttons_Switches_Keyboard:SW_Cherry_MX1A_1.00u_PCB, symbol SW_PUSH
- removed SW3: KEY_3, Buttons_Switches_Keyboard:SW_Cherry_MX1A_1.00u_PCB, symbol SW_PUSH
- removed SW30: KEY_EN, Buttons_Switches_Keyboard:SW_Cherry_MX1A_1.00u_PCB, symbol SW_PUSH
- removed SW31: KEY_CS1, Buttons_Switches_Keyboard:SW_Cherry_MX1A_1.00u_PCB, symbol SW_PUSH
- removed SW32: KEY_Z, Buttons_Switches_Keyboard:SW_Cherry_MX1A_1.00u_PCB, symbol SW_PUSH
- removed SW33: KEY_X, Buttons_Switches_Keyboard:SW_Cherry_MX1A_1.00u_PCB, symbol SW_PUSH
- removed SW34: KEY_C, Buttons_Switches_Keyboard:SW_Cherry_MX1A_1.00u_PCB, symbol SW_PUSH
- removed SW35: KEY_V, Buttons_Switches_Keyboard:SW_Cherry_MX1A_1.00u_PCB, symbol SW_PUSH
- removed SW36: KEY_B, Buttons_Switches_Keyboard:SW_Cherry_MX1A_1.00u_PCB, symbol SW_PUSH
- removed SW37: KEY_N, Buttons_Switches_Keyboard:SW_Cherry_MX1A_1.00u_PCB, symbol SW_PUSH
- removed SW38: KEY_M, Buttons_Switches_Keyboard:SW_Cherry_MX1A_1.00u_PCB, symbol SW_PUSH
- removed SW39: KEY_SS1, Buttons_Switches_Keyboard:SW_Cherry_MX1A_1.00u_PCB, symbol SW_PUSH
- removed SW4: KEY_4, Buttons_Switches_Keyboard:SW_Cherry_MX1A_1.00u_PCB, symbol SW_PUSH
- removed SW40: KEY_SP, Buttons_Switches_Keyboard:SW_Cherry_MX1A_1.00u_PCB, symbol SW_PUSH
- removed SW41: KEY_CS2, Buttons_Switches_Keyboard:SW_Cherry_MX1A_1.00u_PCB, symbol SW_PUSH
- removed SW42: KEY_SS2, Buttons_Switches_Keyboard:SW_Cherry_MX1A_1.00u_PCB, symbol SW_PUSH
- removed SW43: KEY_EDIT, Buttons_Switches_Keyboard:SW_Cherry_MX1A_1.00u_PCB, symbol SW_PUSH
- removed SW44: KEY_CL, Buttons_Switches_Keyboard:SW_Cherry_MX1A_1.00u_PCB, symbol SW_PUSH
- removed SW45: KEY_TV, Buttons_Switches_Keyboard:SW_Cherry_MX1A_1.00u_PCB, symbol SW_PUSH
- removed SW46: KEY_IV, Buttons_Switches_Keyboard:SW_Cherry_MX1A_1.00u_PCB, symbol SW_PUSH
- removed SW47: KEY_LEFT, Buttons_Switches_Keyboard:SW_Cherry_MX1A_1.00u_PCB, symbol SW_PUSH
- removed SW48: KEY_DOWN, Buttons_Switches_Keyboard:SW_Cherry_MX1A_1.00u_PCB, symbol SW_PUSH
- removed SW49: KEY_UP, Buttons_Switches_Keyboard:SW_Cherry_MX1A_1.00u_PCB, symbol SW_PUSH
- removed SW5: KEY_5, Buttons_Switches_Keyboard:SW_Cherry_MX1A_1.00u_PCB, symbol SW_PUSH
- removed SW50: KEY_RIGHT, Buttons_Switches_Keyboard:SW_Cherry_MX1A_1.00u_PCB, symbol SW_PUSH
- removed SW51: KEY_GR, Buttons_Switches_Keyboard:SW_Cherry_MX1A_1.00u_PCB, symbol SW_PUSH
- removed SW52: KEY_DEL, Buttons_Switches_Keyboard:SW_Cherry_MX1A_1.00u_PCB, symbol SW_PUSH
- removed SW53: KEY_QUOT, Buttons_Switches_Keyboard:SW_Cherry_MX1A_1.00u_PCB, symbol SW_PUSH
- removed SW54: KEY_SEM, Buttons_Switches_Keyboard:SW_Cherry_MX1A_1.00u_PCB, symbol SW_PUSH
- removed SW55: KEY_BREAK, Buttons_Switches_Keyboard:SW_Cherry_MX1A_1.00u_PCB, symbol SW_PUSH
- removed SW56: KEY_DOT, Buttons_Switches_Keyboard:SW_Cherry_MX1A_1.00u_PCB, symbol SW_PUSH
- removed SW57: KEY_COMMA, Buttons_Switches_Keyboard:SW_Cherry_MX1A_1.00u_PCB, symbol SW_PUSH
- removed SW58: KEY_EXT, Buttons_Switches_Keyboard:SW_Cherry_MX1A_1.00u_PCB, symbol SW_PUSH
- removed SW6: KEY_6, Buttons_Switches_Keyboard:SW_Cherry_MX1A_1.00u_PCB, symbol SW_PUSH
- removed SW7: KEY_7, Buttons_Switches_Keyboard:SW_Cherry_MX1A_1.00u_PCB, symbol SW_PUSH
- removed SW8: KEY_8, Buttons_Switches_Keyboard:SW_Cherry_MX1A_1.00u_PCB, symbol SW_PUSH
- removed SW9: KEY_9, Buttons_Switches_Keyboard:SW_Cherry_MX1A_1.00u_PCB, symbol SW_PUSH
- added C?: 10uF, Capacitors_Tantalum_SMD:TantalC_SizeC_EIA-6032_HandSoldering, symbol CP
- added P1: CONN_02X17, symbol CONN_02X17
- added P2, P3: CONN_02X20, symbol CONN_02X20
- added P4: CONN_01X02, symbol CONN_01X02
- added R53: 10K, Resistors_SMD:R_0805_HandSoldering, symbol R
- added R54: 1K, Resistors_SMD:R_0805_HandSoldering, symbol R
- added R55: 0R, Resistors_SMD:R_0805_HandSoldering, symbol R
Connections:
- net D0 is gone; now on net KD0: R40.2
- net D1 is gone; now on net KD1: R41.2
- net D2 is gone; now on net KD2: R42.2
- net D3 is gone; now on net KD3: R43.2
- net D4 is gone; now on net KD4: R44.2
- net +3V3: now also R2.1, R3.2, R4.2, R5.2, C?.1, P2.1 (P1), P2.17 (P17), R53.2, R55.1; no longer R2.2, R3.1, R4.1, R5.1
- net GND: now also C?.2, P2.14 (P14), P2.20 (P20), P2.25 (P25), P2.30 (P30), P2.34 (P34), P2.39 (P39), P2.6 (P6), P2.9 (P9), P3.14 (P14), P3.20 (P20), P3.25 (P25), P3.30 (P30), P3.34 (P34), P3.39 (P39), P3.6 (P6), P3.9 (P9), P4.2 (P2)
- net KA10: now also P1.3 (P3)
- net KA11: now also P1.4 (P4)
- net KA12: now also P1.5 (P5)
- net KA13: now also P1.6 (P6)
- net KA14: now also P1.7 (P7)
- net KA15: now also P1.8 (P8)
- net KA8: now also P1.1 (P1)
- net KA9: now also P1.2 (P2)
- net KD0: now also P1.9 (P9); no longer R40.1
- net KD1: now also R2.2, P1.10 (P10); no longer R2.1, R41.1
- net KD2: now also R3.1, P1.11 (P11); no longer R3.2, R42.1
- net KD3: now also R4.1, P1.12 (P12); no longer R4.2, R43.1
- net KD4: now also R5.1, P1.13 (P13); no longer R44.1, R5.2
- net KCL: now reaches D2.2 (A), R8.2, R9.1
- net KCL: now also P1.21 (P21)
- net KTV: now reaches D3.2 (A), R10.2, R11.1
- net KTV: now also P1.23 (P23)
- net KDOWN: now reaches D6.2 (A), R16.2, R17.1
- net KDOWN: now also P1.29 (P29)
- net KUP: now reaches D7.2 (A), R18.2, R19.1
- net KUP: now also P1.31 (P31)
- net KRIGHT: now reaches D8.2 (A), R20.2, R21.1
- net KRIGHT: now also P1.33 (P33)
- net KQUOT: now reaches D11.2 (A), R26.2, R27.1
- net KQUOT: now also P1.22 (P22)
- net KSEM: now reaches D12.2 (A), R28.2, R29.1
- net KSEM: now also P1.24 (P24)
- net KBREAK: now reaches D13.2 (A), R30.2, R31.1
- net KBREAK: now also P1.26 (P26)
- net KIV: now reaches D4.2 (A), R12.2, R13.1
- net KIV: now also P1.25 (P25)
- net KGR: now reaches D9.2 (A), R22.2, R23.1
- net KGR: now also P1.18 (P18)
- net KDOT: now reaches D14.2 (A), R32.2, R33.1
- net KDOT: now also P1.28 (P28)
- net KLEFT: now reaches D5.2 (A), R14.2, R15.1
- net KLEFT: now also P1.27 (P27)
- net KDEL: now reaches D10.2 (A), R24.2, R25.1
- net KDEL: now also P1.20 (P20)
- net KCOMMA: now reaches D15.2 (A), R34.2, R35.1
- net KCOMMA: now also P1.30 (P30)
- net KEDIT: now reaches D1.2 (A), R6.2, R7.1
- net KEDIT: now also P1.19 (P19)
- net KEXT: now reaches D16.2 (A), D17.2 (A)
- net KEXT: now also P1.32 (P32)
- net A10 renamed GPIO6
- net GPIO6: now also P2.31 (P31)
- net A11 renamed GPIO7
- net GPIO7: now also P2.26 (P26)
- net A12 renamed GPIO8
- net GPIO8: now also P2.24 (P24)
- net A13 renamed GPIO9
- net GPIO9: now also P2.21 (P21)
- net A14 renamed GPIO10
- net GPIO10: now also P2.19 (P19)
- net A15 renamed GPIO11
- net GPIO11: now also P2.23 (P23)
- net A8 renamed GPIO4
- net GPIO4: now also P2.7 (P7)
- net A9 renamed GPIO5
- net GPIO5: now also P2.29 (P29)
- new net: P4.1 (P1), R53.1, R54.1
- new net GPIO12: P2.32 (P32), R40.1
- new net GPIO13: P2.33 (P33), R41.1
- new net GPIO14: P2.8 (P8), R42.1
- new net GPIO15: P2.10 (P10), R43.1
- new net GPIO16: P2.36 (P36), R44.1
- new net GPIO17: P2.11 (P11), R54.2
- new net GPIO18: P2.12 (P12), P3.12 (P12)
- new net GPIO19: P2.35 (P35), P3.35 (P35)
- new net GPIO2: P2.3 (P3), P3.3 (P3)
- new net GPIO20: P2.38 (P38), P3.38 (P38)
- new net GPIO21: P2.40 (P40), P3.40 (P40)
- new net GPIO22: P2.15 (P15)
- new net GPIO23: P2.16 (P16)
- new net GPIO24: P2.18 (P18)
- new net GPIO25: P2.22 (P22)
- new net GPIO26: P2.37 (P37), P3.37 (P37)
- new net GPIO27: P2.13 (P13)
- new net GPIO3: P2.5 (P5), P3.5 (P5)
- new net ID_SC: P2.28 (P28)
- new net ID_SD: P2.27 (P27)
- new net KCOMM: P1.17 (P17), R55.2
- new net VCC_5V: P2.2 (P2), P2.4 (P4), P3.2 (P2), P3.4 (P4)
- no-connect marks 1 -> 34
Other:
- note added: "HiFi Berry+"
- note added: "Keyboard"
- note added: "Raspberry Pi"
- note added: "Reset"
- moved on the sheet: C1, Q1, Q2, Q3, Q4, Q5, Q6, Q7, Q8, R1, R2, R3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

Commit message: pcb
Parts:
- gave numbers to parts that had none: 1
Connections:
- net +3V3: no longer C2.1
- net VCC_5V renamed +5V
- net +5V: now also C2.1
Other:
- moved on the sheet: C1, C2, P3, P4, R53, R54

Commit message: pcb
Parts:
- added P5: CONN_01X02, Connectors_Phoenix:PhoenixContact_MCV-G_02x5.08mm_Vertical, symbol CONN_01X02
- P1: footprint (none) -> Pin_Headers:Pin_Header_Angled_2x17
- P2, P3: footprint (none) -> Pin_Headers:Pin_Header_Angled_2x20
- P4: footprint (none) -> Pin_Headers:Pin_Header_Angled_1x02
Connections:
- net +5V: now also P5.1 (P1)
- net GND: now also P5.2 (P2)
Changed lines of the file:
@@
 F 0 "P1" H 1700 2750 50  0000 C CNN
 F 1 "CONN_02X17" V 1700 1850 50  0000 C CNN
-F 2 "" H 1700 750 50  0000 C CNN
+F 2 "Pin_Headers:Pin_Header_Angled_2x17" H 1700 750 50  0001 C CNN
 F 3 "" H 1700 750 50  0000 C CNN
 	1    1700 1850
@@
 F 0 "P2" H 3750 3050 50  0000 C CNN
 F 1 "CONN_02X20" V 3750 2000 50  0000 C CNN
-F 2 "" H 3750 1050 50  0000 C CNN
+F 2 "Pin_Headers:Pin_Header_Angled_2x20" H 3750 1050 50  0001 C CNN
 F 3 "" H 3750 1050 50  0000 C CNN
 	1    3750 2000
@@
 F 0 "P3" H 5700 3050 50  0000 C CNN
 F 1 "CONN_02X20" V 5700 2000 50  0000 C CNN
-F 2 "" H 5700 1050 50  0000 C CNN
+F 2 "Pin_Headers:Pin_Header_Angled_2x20" H 5700 1050 50  0001 C CNN
 F 3 "" H 5700 1050 50  0000 C CNN
 	1    5700 2000
@@
 F 0 "P4" H 7850 3100 50  0000 C CNN
 F 1 "CONN_01X02" V 7950 2950 50  0000 C CNN
-F 2 "" H 7850 2950 50  0000 C CNN
+F 2 "Pin_Headers:Pin_Header_Angled_1x02" H 7850 2950 50  0001 C CNN
 F 3 "" H 7850 2950 50  0000 C CNN
 	1    7850 2950
@@
 Connection ~ 7600 1800
 Wire Wire Line
-	7200 1800 7950 1800
+	7200 1800 8300 1800
 Connection ~ 7600 1400
 Wire Wire Line
@@
 Wire Wire Line
 	6600 1050 5950 1050
+$Comp
+L CONN_01X02 P5
+U 1 1 5B11089A
+P 8500 1750
+F 0 "P5" H 8500 1900 50  0000 C CNN
+F 1 "CONN_01X02" V 8600 1750 50  0000 C CNN
+F 2 "Connectors_Phoenix:PhoenixContact_MCV-G_02x5.08mm_Vertical" H 8500 1750 50  0001 C CNN
+F 3 "" H 8500 1750 50  0000 C CNN
+	1    8500 1750
+	1    0    0    -1
+$EndComp
+Connection ~ 7950 1800
+Wire Wire Line
+	8300 1400 8300 1700
+Connection ~ 8300 1400
 $EndSCHEMATC

Commit message: pcb
Parts:
- removed R55: 0R, Resistors_SMD:R_0805_HandSoldering, symbol R
Connections:
- net KCOMM is gone; now on net +3V3: P1.17 (P17)
- net +3V3: now also P1.15 (P15), P1.16 (P16)
- no-connect marks 34 -> 32
Changed lines of the file:
@@
 Text Label 850  1650 0    60   ~ 0
 KD4
-NoConn ~ 1450 1750
-NoConn ~ 1950 1750
-NoConn ~ 1950 1650
 NoConn ~ 1950 2650
 Text Label 850  1850 0    60   ~ 0
-KCOMM
+VCC
 Text Label 850  1950 0    60   ~ 0
 KEDIT
@@
 Entry Wire Line
 	6300 6100 6400 6200
-$Comp
-L R R55
-U 1 1 5B31AEEB
-P 10250 2750
-F 0 "R55" V 10330 2750 50  0000 C CNN
-F 1 "0R" V 10250 2750 50  0000 C CNN
-F 2 "Resistors_SMD:R_0805_HandSoldering" V 10180 2750 50  0001 C CNN
-F 3 "" H 10250 2750 50  0000 C CNN
-	1    10250 2750
-	0    1    1    0
-$EndComp
-Wire Wire Line
-	10100 2750 8950 2750
-Wire Wire Line
-	10400 2750 11100 2750
-Entry Wire Line
-	11100 2750 11200 2850
-Entry Wire Line
-	8850 2650 8950 2750
-Text Label 8950 2750 0    60   ~ 0
-KCOMM
-Text Label 10750 2750 0    60   ~ 0
-VCC
 NoConn ~ 5950 1450
 NoConn ~ 2750 1650
@@
 	8300 1400 8300 1700
 Connection ~ 8300 1400
+Wire Wire Line
+	1450 1750 1350 1750
+Wire Wire Line
+	1350 1750 1350 1850
+Connection ~ 1350 1850
+Wire Wire Line
+	1950 1750 2550 1750
+Entry Wire Line
+	2550 1750 2650 1850
+Text Label 2150 1750 0    60   ~ 0
+VCC
+NoConn ~ 1950 1650
 $EndSCHEMATC
