File: keyboard/zx_keyboard.kicad_pcb (KiCad board)
At the start: 2 copper layers, 257 x 95 mm, 59 parts, among them P1 CONN_02X17, SW1 KEY_1, SW10 KEY_0, SW11 KEY_Q, SW12 KEY_W, SW13 KEY_E, SW14 KEY_R, SW15 KEY_T, SW16 KEY_Y, SW17 KEY_U, SW18 KEY_I, SW19 KEY_O, SW2 KEY_2, SW20 KEY_P, SW21 KEY_A, SW22 KEY_S, SW23 KEY_D, SW24 KEY_F, SW25 KEY_G, SW26 KEY_H, SW27 KEY_J, SW28 KEY_K, SW29 KEY_L, SW3 KEY_3, SW30 KEY_EN, SW31 KEY_CS1, SW32 KEY_Z, SW33 KEY_X, SW34 KEY_C, SW35 KEY_V, SW36 KEY_B, SW37 KEY_N, SW38 KEY_M, SW39 KEY_SS1, SW4 KEY_4, SW40 KEY_SP, SW41 KEY_CS2, SW42 KEY_SS2, SW43 KEY_EDIT, SW44 KEY_CL, SW45 KEY_TV, SW46 KEY_IV, SW47 KEY_LEFT, SW48 KEY_DOWN, SW49 KEY_UP, SW5 KEY_5, SW50 KEY_RIGHT, SW51 KEY_GR, SW52 KEY_DEL, SW53 KEY_QUOT, SW54 KEY_SEM, SW55 KEY_BREAK, SW56 KEY_DOT, SW57 KEY_COMMA, SW58 KEY_EXT, SW6 KEY_6, SW7 KEY_7, SW8 KEY_8, SW9 KEY_9

Commit message: zx
Parts:
- moved SW11 33.9 mm to (78.1, 77.2)
- moved SW12 33.9 mm to (97.1, 77.2)
- moved SW13 33.9 mm to (116.1, 77.2)
- moved SW14 33.9 mm to (135.1, 77.2)
- moved SW15 33.9 mm to (154.1, 77.2)
- moved SW16 33.9 mm to (173.1, 77.2)
- moved SW17 33.9 mm to (192.1, 77.2)
- moved SW18 33.9 mm to (211.1, 77.2)
- moved SW19 33.9 mm to (230.1, 77.2)
- moved SW20 33.9 mm to (249.1, 77.2)
- moved SW51 33.9 mm to (59.1, 77.2)
- moved P1 33.8 mm to (120.8, 35.3)
- moved SW1 33.8 mm to (68.8, 58.2)
- moved SW10 33.8 mm to (239.8, 58.2)
- moved SW2 33.8 mm to (87.8, 58.2)
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Other:
- board size 257 x 95 mm -> 257 x 127 mm
- net class Default: clearance 0.2 -> 0.5; trace_width 0.25 -> 0.5
- rule trace_clearance: 0.2 -> 0.5
- rule trace_min: 0.2 -> 0.5
- board text added: "ZX Keyboard v0.1"

Commit message: pcb
Parts:
- added REF**: R_1206_HandSoldering, Resistors_SMD:R_1206_HandSoldering, B.Cu at (257.8, 86.4)
Routing:
- net /KA15: track 0.00 -> 387.5 mm
- net /KCOMM: track 0.00 -> 308.9 mm
- net /KA8: track 0.00 -> 219.4 mm
- net /KIV: track 0.00 -> 151.6 mm
- net /KBREAK: track 0.00 -> 147.0 mm
- net /KD0: track 0.00 -> 127.7 mm
- net /KD4: track 0.00 -> 102.1 mm
- net /KA14: track 0.00 -> 97.1 mm
- net /KA13: track 0.00 -> 76.0 mm
- net /KA12: track 0.00 -> 76.0 mm
- net /KA11: track 0.00 -> 76.0 mm
- net /KA9: track 0.00 -> 76.0 mm
- net /KA10: track 0.00 -> 76.0 mm

Commit message: pcb
Parts:
- removed REF**: R_1206_HandSoldering, Resistors_SMD:R_1206_HandSoldering
Routing:
- net /KD3: track 0.00 -> 252.9 mm, vias 0 -> 12
- net /KD0: track 127.7 -> 332.8 mm, vias 0 -> 2
- net /KIV: track 151.6 -> 0.00 mm
- net /KD4: track 102.1 -> 227.7 mm, vias 0 -> 4
- net /KCOMM: track 308.9 -> 419.5 mm
- net /KD1: track 0.00 -> 108.0 mm, vias 0 -> 2
- net /KGR: track 0.00 -> 93.1 mm
- net /KD2: track 0.00 -> 86.6 mm, vias 0 -> 4
- net /KDEL: track 0.00 -> 83.3 mm
- net /KQUOT: track 0.00 -> 77.0 mm
- net /KSEM: track 0.00 -> 70.6 mm
- net /KA13: track 76.0 -> 138.7 mm
- net /KA12: track 76.0 -> 136.6 mm, vias 0 -> 2
- net /KA15: track 387.5 -> 447.0 mm, vias 0 -> 2
- net /KDOT: track 0.00 -> 57.8 mm
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Other:
- net class Default: via_dia 0.6 -> 2; via_drill 0.4 -> 0.01
- rule via_min_drill: 0.3 -> 0.01
- rule via_min_size: 0.4 -> 2

Commit message: pcb
Parts:
- moved P1 48.4 mm to (74.5, 49.5)
Routing:
- net /KD1: track 108.0 -> 562.9 mm, vias 2 -> 26
- net /KD2: track 86.6 -> 329.1 mm, vias 4 -> 22
- net /KA14: track 97.1 -> 278.3 mm, vias 0 -> 18
- net /KD0: track 332.8 -> 509.2 mm, vias 2 -> 26
- net /KA15: track 447.0 -> 595.4 mm, vias 2 -> 24
- net /KBREAK: track 146.6 -> 8.22 mm, vias 0 -> 1
- net /KCOMM: track 419.5 -> 547.6 mm, vias 0 -> 12
- net /KA8: track 219.4 -> 324.5 mm, vias 0 -> 12
- net /KGR: track 93.1 -> 7.41 mm, vias 0 -> 1
- net /KA9: track 126.0 -> 202.4 mm, vias 0 -> 10
- net /KDEL: track 83.3 -> 7.48 mm, vias 0 -> 1
- net /KA13: track 138.7 -> 210.6 mm, vias 0 -> 6
- net /KQUOT: track 77.0 -> 7.15 mm, vias 0 -> 1
- net /KSEM: track 70.6 -> 7.48 mm, vias 0 -> 1
- net /KD3: track 252.9 -> 313.8 mm, vias 12 -> 16
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Other:
- board size 257 x 127 mm -> 257 x 111 mm
- net class ext_pads added: clearance 1.25, trace_width 1.27, via_dia 2, via_drill 0.01

Commit message: pcb
Routing:
- net /KD4: track 270.7 -> 301.4 mm, vias 8 -> 6
- net /KD0: track 509.2 -> 538.0 mm, vias 26 -> 12
- net /KA12: track 189.3 -> 211.0 mm, vias 10 -> 6
- net /KCOMM: track 547.6 -> 530.7 mm, vias 12 -> 6
- net /KA14: track 278.3 -> 268.3 mm, vias 18 -> 10
- net /KD3: track 313.8 -> 321.5 mm, vias 16 -> 10
- net /KD2: track 329.1 -> 325.9 mm, vias 22 -> 20
- net /KA13: track 210.6 -> 213.4 mm
- net /KA9: track 202.4 -> 199.7 mm, vias 10 -> 8
- net /KD1: track 562.9 -> 565.5 mm, vias 26 -> 12
- net /KA15: track 595.4 -> 593.5 mm, vias 24 -> 16
- net /KA11: track 105.9 -> 107.4 mm
- net /KA10: track 115.1 -> 113.9 mm
Other:
- net class Default: trace_width 0.5 -> 0.8
- rule trace_min: 0.5 -> 0.8

Commit message: pcb
Routing:
- net /KD0: track 538.0 -> 514.9 mm
- net /KD2: track 325.9 -> 305.5 mm, vias 20 -> 16
- net /KD1: track 565.5 -> 552.2 mm, vias 12 -> 14
- net /KA15: track 593.5 -> 604.0 mm, vias 16 -> 12
- net /KA9: track 199.7 -> 191.8 mm, vias 8 -> 6
- net /KD3: track 321.5 -> 328.3 mm, vias 10 -> 12
- net /KA14: track 268.3 -> 271.6 mm, vias 10 -> 6
- net /KCOMM: track 530.7 -> 527.7 mm
- net /KA13: track 213.4 -> 215.0 mm

Commit message: keyboard pcb
Routing:
- net /KA8: track 324.5 -> 332.3 mm
- net /KD1: track 552.2 -> 545.5 mm
- net /KA15: track 604.0 -> 610.4 mm
- net /KD0: track 514.9 -> 521.0 mm
- added copper zone on B.Cu, net (none)
