File: keyboard/zx_keyboard.kicad_pcb (KiCad board)
At the start: 2 copper layers, 257 x 111 mm, 59 parts, among them P1 CONN_02X17, SW1 KEY_1, SW10 KEY_0, SW11 KEY_Q, SW12 KEY_W, SW13 KEY_E, SW14 KEY_R, SW15 KEY_T, SW16 KEY_Y, SW17 KEY_U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

Commit message: TV<->IV fix
Parts:
- moved SW45 19.0 mm to (30.8, 58.2)
- moved SW46 19.0 mm to (49.8, 58.2)
Routing:
- net /KTV: track 8.61 -> 6.81 mm
- net /KIV: track 6.81 -> 8.61 mm
